Commit message: Modify valkyrie URDF to use .obj meshes

File: examples/valkyrie/urdf/urdf/valkyrie_A_sim_drake_one_neck_dof_wide_ankle_rom.urdf (robot description, URDF)
Before this commit: robot valkyrie, 87 links, 86 joints
Links:
- link leftAnklePitchLink: geometry collision mesh filename=package://valkyrie/urdf/model/meshes/legs/lj5.obj; visual mesh filename=package://valkyrie/urdf/model/meshes/legs/lj5.obj
- link leftElbowPitchLink: geometry collision mesh filename=package://valkyrie/urdf/model/meshes/arms/aj4_left.obj; visual mesh filename=package://valkyrie/urdf/model/meshes/arms/aj4_left.obj
- link leftFoot: geometry collision box size=0.27 0.16 0.064; collision sphere radius=0.0
- link leftForearmLink: geometry collision mesh filename=package://valkyrie/urdf/model/meshes/arms/aj5_left.obj; visual mesh filename=package://valkyrie/urdf/model/meshes/arms/aj5_left.obj
- link leftHipPitchLink: geometry collision mesh filename=package://valkyrie/urdf/model/meshes/legs/lj3_left.obj; visual mesh filename=package://valkyrie/urdf/model/meshes/legs/lj3_left.obj
- link leftHipRollLink: geometry collision mesh filename=package://valkyrie/urdf/model/meshes/legs/lj2_left.obj; visual mesh filename=package://valkyrie/urdf/model/meshes/legs/lj2_left.obj
- link leftHipYawLink: geometry collision mesh filename=package://valkyrie/urdf/model/meshes/legs/lj1_left.obj; visual mesh filename=package://valkyrie/urdf/model/meshes/legs/lj1_left.obj
- link leftIndexFingerPitch1Link: geometry collision mesh filename=package://valkyrie/urdf/model/meshes/fingers/indexj1_left.o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; visual mesh filename=package://valkyrie/urdf/model/meshes/fingers/indexj1_left.o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
- link leftIndexFingerPitch2Link: geometry collision mesh filename=package://valkyrie/urdf/model/meshes/fingers/indexj2_left.o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; visual mesh filename=package://valkyrie/urdf/model/meshes/fingers/indexj2_left.o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
- link leftIndexFingerPitch3Link: geometry collision mesh filename=package://valkyrie/urdf/model/meshes/fingers/indexj3_left.o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; visual mesh filename=package://valkyrie/urdf/model/meshes/fingers/indexj3_left.o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
- link leftKneePitchLink: geometry collision mesh filename=package://valkyrie/urdf/model/meshes/legs/lj4_left.obj; visual mesh filename=package://valkyrie/urdf/model/meshes/legs/lj4_left.obj
- link leftPalm: geometry collision mesh filename=package://valkyrie/urdf/model/meshes/arms/palm_left.obj; visual mesh filename=package://valkyrie/urdf/model/meshes/arms/palm_left.obj
- link leftPinkyPitch1Link: geometry collision mesh filename=package://valkyrie/urdf/model/meshes/fingers/pinkyj1_left.o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; visual mesh filename=package://valkyrie/urdf/model/meshes/fingers/pinkyj1_left.o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
- link leftPinkyPitch2Link: geometry collision mesh filename=package://valkyrie/urdf/model/meshes/fingers/pinkyj2_left.o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; visual mesh filename=package://valkyrie/urdf/model/meshes/fingers/pinkyj2_left.o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
- link leftPinkyPitch3Link: geometry collision mesh filename=package://valkyrie/urdf/model/meshes/fingers/pinkyj3_left.o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; visual mesh filename=package://valkyrie/urdf/model/meshes/fingers/pinkyj3_left.o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
- link leftShoulderPitchLink: geometry collision mesh filename=package://valkyrie/urdf/model/meshes/arms/aj1_left.obj; visual mesh filename=package://valkyrie/urdf/model/meshes/arms/aj1_left.obj
- link leftShoulderRollLink: geometry collision mesh filename=package://valkyrie/urdf/model/meshes/arms/aj2_left.obj; visual mesh filename=package://valkyrie/urdf/model/meshes/arms/aj2_left.obj
- link leftShoulderYawLink: geometry collision mesh filename=package://valkyrie/urdf/model/meshes/arms/aj3_left.obj; visual mesh filename=package://valkyrie/urdf/model/meshes/arms/aj3_left.obj
- link leftThumbPitch1Link: geometry collision mesh filename=package://valkyrie/urdf/model/meshes/fingers/thumbj2_left.o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; visual mesh filename=package://valkyrie/urdf/model/meshes/fingers/thumbj2_left.o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
- link leftThumbPitch2Link: geometry collision mesh filename=package://valkyrie/urdf/model/meshes/fingers/thumbj3_left.o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; visual mesh filename=package://valkyrie/urdf/model/meshes/fingers/thumbj3_left.o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
- link leftThumbPitch3Link: geometry collision mesh filename=package://valkyrie/urdf/model/meshes/fingers/thumbj4_left.o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; visual mesh filename=package://valkyrie/urdf/model/meshes/fingers/thumbj4_left.o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
- link leftThumbRollLink: geometry collision mesh filename=package://valkyrie/urdf/model/meshes/fingers/thumbj1_left.o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; visual mesh filename=package://valkyrie/urdf/model/meshes/fingers/thumbj1_left.o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
- link leftWristRollLink: geometry collision mesh filename=package://valkyrie/urdf/model/meshes/arms/aj6_left.obj; visual mesh filename=package://valkyrie/urdf/model/meshes/arms/aj6_left.obj
- link lowerNeckPitchLink: geometry collision mesh filename=package://valkyrie/urdf/model/meshes/head/neckj1.obj; visual mesh filename=package://valkyrie/urdf/model/meshes/head/neckj1.obj
- link neckYawLink: geometry collision mesh filename=package://valkyrie/urdf/model/meshes/head/neckj2.obj; visual mesh filename=package://valkyrie/urdf/model/meshes/head/neckj2.obj
- link pelvis: geometry collision mesh filename=package://valkyrie/urdf/model/meshes/pelvis/pelvis.obj; visual mesh filename=package://valkyrie/urdf/model/meshes/pelvis/pelvis.obj
- link rightAnklePitchLink: geometry collision mesh filename=package://valkyrie/urdf/model/meshes/legs/lj5.obj; visual mesh filename=package://valkyrie/urdf/model/meshes/legs/lj5.obj
- link rightElbowPitchLink: geometry collision mesh filename=package://valkyrie/urdf/model/meshes/arms/aj4_right.obj; visual mesh filename=package://valkyrie/urdf/model/meshes/arms/aj4_right.obj
- link rightFoot: geometry collision box size=0.27 0.16 0.064; collision sphere radius=0.0
- link rightForearmLink: geometry collision mesh filename=package://valkyrie/urdf/model/meshes/arms/aj5_right.obj; visual mesh filename=package://valkyrie/urdf/model/meshes/arms/aj5_right.obj
- link rightHipPitchLink: geometry collision mesh filename=package://valkyrie/urdf/model/meshes/legs/lj3_right.obj; visual mesh filename=package://valkyrie/urdf/model/meshes/legs/lj3_right.obj
- link rightHipRollLink: geometry collision mesh filename=package://valkyrie/urdf/model/meshes/legs/lj2_right.obj; visual mesh filename=package://valkyrie/urdf/model/meshes/legs/lj2_right.obj
- link rightHipYawLink: geometry collision mesh filename=package://valkyrie/urdf/model/meshes/legs/lj1_right.obj; visual mesh filename=package://valkyrie/urdf/model/meshes/legs/lj1_right.obj
- link rightKneePitchLink: geometry collision mesh filename=package://valkyrie/urdf/model/meshes/legs/lj4_right.obj; visual mesh filename=package://valkyrie/urdf/model/meshes/legs/lj4_right.obj
- link rightPalm: geometry collision mesh filename=package://valkyrie/urdf/model/meshes/arms/palm_right.obj; visual mesh filename=package://valkyrie/urdf/model/meshes/arms/palm_right.obj
- link rightShoulderPitchLink: geometry collision mesh filename=package://valkyrie/urdf/model/meshes/arms/aj1_right.obj; visual mesh filename=package://valkyrie/urdf/model/meshes/arms/aj1_right.obj
- link rightShoulderRollLink: geometry collision mesh filename=package://valkyrie/urdf/model/meshes/arms/aj2_right.obj; visual mesh filename=package://valkyrie/urdf/model/meshes/arms/aj2_right.obj
- link rightShoulderYawLink: geometry collision mesh filename=package://valkyrie/urdf/model/meshes/arms/aj3_right.obj; visual mesh filename=package://valkyrie/urdf/model/meshes/arms/aj3_right.obj
- link rightWristRollLink: geometry collision mesh filename=package://valkyrie/urdf/model/meshes/arms/aj6_right.obj; visual mesh filename=package://valkyrie/urdf/model/meshes/arms/aj6_right.obj
- link torso: geometry collision mesh filename=package://valkyrie/urdf/model/meshes/torso/torso.obj; visual mesh filename=package://valkyrie/urdf/model/meshes/torso/torso.obj
- link torsoPitchLink: geometry collision mesh filename=package://valkyrie/urdf/model/meshes/torso/torsopitch.obj; visual mesh filename=package://valkyrie/urdf/model/meshes/torso/torsopitch.obj
- link torsoYawLink: geometry collision mesh filename=package://valkyrie/urdf/model/meshes/torso/torsoyaw.obj; visual mesh filename=package://valkyrie/urdf/model/meshes/torso/torsoyaw.obj
